File: RadioHAT_Card_SX1280_Dual_Channel/RadioHAT_Card_SX1280_Dual_Channel.kicad_pcb (KiCad board)
At the start: 2 copper layers, 30 x 51 mm, 9 parts, among them J2 Conn_Coaxial, J3 Conn_Coaxial

Commit message: Minor cleanup
Routing:
- net NSS0: track 67.8 -> 68.7 mm
- net GND: vias 28 -> 29
