File: RadioHAT_Card_Dorji/RadioHAT_Card_Dorji.kicad_pcb (KiCad board)
At the start: 2 copper layers, 30 x 51 mm, 10 parts, among them J2 Conn_Coaxial, J3 Conn_Coaxial, J4 Conn_Coaxial, J5 Conn_Coaxial, J6 Conn_Coaxial

Commit message: [PCB] Make cards' githash variable
Other:
- board text added: "Dorji rev. A gitrev ${GITHASH}"
- board text removed: "Dorji rev. A gitrev GITHASH"
Changed lines of the file:
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@@
 		)
 	)
-	(gr_text "Dorji rev. A\ngitrev GITHASH"
+	(gr_text "Dorji rev. A\ngitrev ${GITHASH}"
 		(at 132.8 71.7 0)
 		(layer "F.Cu")

Commit message: Update symbols to align with library
Connections:
- J1 pad 20: (no net) -> unconnected-(J1-NSS1-Pad20)
- J1 pad 28: (no net) -> unconnected-(J1-5V-Pad28)
- J1 pad 48: (no net) -> unconnected-(J1-5V-Pad48)
- J1 pad 6: (no net) -> unconnected-(J1-5V-Pad6)
Changed lines of the file:
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@@
 		)
 	)
+	(property "GITHASH" "GITHASH")
 	(net 0 "")
 	(net 1 "GND")
@@
 	(net 32 "Net-(J5-Ext)")
 	(net 33 "Net-(J6-Ext)")
+	(net 34 "unconnected-(J1-5V-Pad28)")
+	(net 35 "unconnected-(J1-5V-Pad6)")
+	(net 36 "unconnected-(J1-NSS1-Pad20)")
+	(net 37 "unconnected-(J1-5V-Pad48)")
 	(footprint "RadioHAT:Mini_PCIe_Full"
 		(layer "F.Cu")
@@
 			)
 		)
+		(property "Mouser" "571-1775838-2"
+			(at 0 0 0)
+			(unlocked yes)
+			(layer "F.Fab")
+			(hide yes)
+			(effects
+				(font
+					(size 1 1)
+					(thickness 0.15)
+				)
+			)
+		)
 		(sheetname "/")
 		(sheetfile "RadioHAT_Card_Dorji.kicad_sch")
@@
 			(size 2.3 0.6)
 			(layers "B.Cu" "B.Mask" "B.Paste")
+			(net 35 "unconnected-(J1-5V-Pad6)")
+			(pinfunction "5V")
+			(pintype "power_in+no_connect")
 			(thermal_bridge_angle 0)
 		)
@@
 			(size 2.3 0.6)
 			(layers "B.Cu" "B.Mask" "B.Paste")
+			(net 36 "unconnected-(J1-NSS1-Pad20)")
+			(pinfunction "NSS1")
+			(pintype "bidirectional+no_connect")
 			(thermal_bridge_angle 0)
 		)
@@
 			(size 2.3 0.6)
 			(layers "B.Cu" "B.Mask" "B.Paste")
+			(net 34 "unconnected-(J1-5V-Pad28)")
+			(pinfunction "5V")
+			(pintype "power_in+no_connect")
 			(thermal_bridge_angle 0)
 		)
@@
 			(size 2.3 0.6)
 			(layers "B.Cu" "B.Mask" "B.Paste")
+			(net 37 "unconnected-(J1-5V-Pad48)")
+			(pinfunction "5V")
+			(pintype "power_in+no_connect")
 			(thermal_bridge_angle 0)
 		)
@@
 			(layers "F.Cu" "F.Mask" "F.Paste")
 			(net 5 "NSS")
-			(pinfunction "SPI_NSS")
+			(pinfunction "NSS0")
 			(pintype "bidirectional")
 			(thermal_bridge_angle 0)
